File: hardware/kicad_thermo_ctrl/kicad_thermo_ctrl.kicad_pcb (KiCad board)
At the start: 2 copper layers, 68.6 x 53.3 mm, 23 parts, among them P1 Power, P2 Analog, P3 Digital, P4 Digital, P5 CONN_01X01, P6 CONN_01X01, P7 CONN_01X01, P8 CONN_01X01

Commit message: ...
Parts:
- added i2c1: I2C, Connector_PinHeader_2.54mm:PinHeader_1x04_P2.54mm_Vertical, F.Cu at (164.6, 120.0)
- added power_ctrl1: Conn_01x02, TerminalBlock:TerminalBlock_Altech_AK300-2_P5.00mm, F.Cu at (136.4, 87.0)
- moved R_E_L7 10.3 mm to (159.3, 86.2), turned to 180 degrees
- moved L5 8.29 mm to (144.8, 95.9)
- moved L6 8.29 mm to (152.4, 95.9)
- moved L7 8.29 mm to (160.0, 95.9)
- moved T_L5 8.29 mm to (144.8, 91.6)
- moved T_L6 8.29 mm to (152.4, 91.6)
- moved T_L7 8.29 mm to (160.0, 91.6)
- moved R_E_L5 8.10 mm to (144.1, 86.2), turned to 180 degrees
- moved R_E_L6 8.10 mm to (151.7, 86.2), turned to 180 degrees
Routing:
- net +5V: track 33.4 -> 108.5 mm
- net /8: track 0.00 -> 25.0 mm
- net Net-(R_B_L7-Pad1): track 69.9 -> 62.2 mm
- net Net-(R_B_L5-Pad1): track 38.5 -> 31.1 mm
- net Net-(R_B_L6-Pad1): track 63.0 -> 56.0 mm
- net /A5(SCL): track 0.00 -> 4.76 mm
- net /A4(SDA): track 0.00 -> 4.76 mm
- net Net-(R_E_L7-Pad1): track 3.67 -> 3.05 mm
Other:
- board text added: "Thermo_Ctrl Lucas Seara Manoel ls.manoel@gmail.com"
