File: hardware/kicad_thermo_ctrl/kicad_thermo_ctrl.sch (KiCad schematic (older format))
At the start: 23 parts, among them P1 Power, P2 Analog, P3 Digital, P4 Digital, P5 CONN_01X01, P6 CONN_01X01, P7 CONN_01X01, P8 CONN_01X01

Commit message: pcb ok
Parts:
- added i2c1: I2C, Connector_PinHeader_2.54mm:PinHeader_1x04_P2.54mm_Vertical, symbol Connector_Generic:Conn_01x04
- added power_ctrl1: Conn_01x02, TerminalBlock:TerminalBlock_Altech_AK300-2_P5.00mm, symbol Connector_Generic:Conn_01x02
- MAX6675: footprint Connector_PinHeader_2.00mm:PinHeader_1x05_P2.00mm_Vertical -> Connector_PinHeader_2.54mm:PinHeader_1x05_P2.54mm_Vertical
- renumbered NTC_IN to NTC_IN1, R_NTC to R_NTC1
Connections:
- net +5V: now also i2c1.2 (Pin_2)
- net 8: now also power_ctrl1.1 (Pin_1)
- net A4(SDA): now also i2c1.3 (Pin_3)
- net A5(SCL): now also i2c1.4 (Pin_4)
- net GND: now also i2c1.1 (Pin_1), power_ctrl1.2 (Pin_2)
Changed lines of the file:
@@
 EELAYER 30 0
 EELAYER END
-$Descr A4 11693 8268
+$Descr A1 33110 23386
 encoding utf-8
 Sheet 1 1
@@
 	10700 1000 10700 500
 $Comp
-L Device:R R_NTC
+L Device:R R_NTC1
 U 1 1 5E1AB9D1
 P 7550 2900
-F 0 "R_NTC" H 7620 2946 50  0000 L CNN
+F 0 "R_NTC1" H 7620 2946 50  0000 L CNN
 F 1 "10 k" H 7620 2855 50  0000 L CNN
 F 2 "Resistor_SMD:R_0805_2012Metric" V 7480 2900 50  0001 C CNN
@@
 $EndComp
 $Comp
-L power:GND #PWR?
+L power:GND #PWR0101
 U 1 1 5E1B4A8D
 P 7550 3200
-F 0 "#PWR?" H 7550 2950 50  0001 C CNN
+F 0 "#PWR0101" H 7550 2950 50  0001 C CNN
 F 1 "GND" H 7555 3027 50  0000 C CNN
 F 2 "" H 7550 3200 50  0001 C CNN
@@
 $EndComp
 $Comp
-L power:+5V #PWR?
+L power:+5V #PWR0102
 U 1 1 5E1B5326
 P 7550 2150
-F 0 "#PWR?" H 7550 2000 50  0001 C CNN
+F 0 "#PWR0102" H 7550 2000 50  0001 C CNN
 F 1 "+5V" H 7565 2323 50  0000 C CNN
 F 2 "" H 7550 2150 50  0001 C CNN
@@
 $EndComp
 $Comp
-L Connector_Generic:Conn_01x02 NTC_IN
+L Connector_Generic:Conn_01x02 NTC_IN1
 U 1 1 5E1B65E2
 P 7200 2500
-F 0 "NTC_IN" H 7118 2175 50  0000 C CNN
+F 0 "NTC_IN1" H 7118 2175 50  0000 C CNN
 F 1 "Conn_01x02" H 7118 2266 50  0000 C CNN
 F 2 "TerminalBlock:TerminalBlock_Altech_AK300-2_P5.00mm" H 7200 2500 50  0001 C CNN
@@
 $EndComp
 $Comp
-L power:+5V #PWR?
+L power:+5V #PWR0103
 U 1 1 5E1DD58A
 P 2550 1000
-F 0 "#PWR?" H 2550 850 50  0001 C CNN
+F 0 "#PWR0103" H 2550 850 50  0001 C CNN
 F 1 "+5V" H 2565 1173 50  0000 C CNN
 F 2 "" H 2550 1000 50  0001 C CNN
@@
 $EndComp
 $Comp
-L power:GND #PWR?
+L power:GND #PWR0104
 U 1 1 5E1DD596
 P 2550 2450
-F 0 "#PWR?" H 2550 2200 50  0001 C CNN
+F 0 "#PWR0104" H 2550 2200 50  0001 C CNN
 F 1 "GND" H 2555 2277 50  0000 C CNN
 F 2 "" H 2550 2450 50  0001 C CNN
@@
 $EndComp
 $Comp
-L power:+5V #PWR?
+L power:+5V #PWR0105
 U 1 1 5E245901
 P 4450 1000
-F 0 "#PWR?" H 4450 850 50  0001 C CNN
+F 0 "#PWR0105" H 4450 850 50  0001 C CNN
 F 1 "+5V" H 4465 1173 50  0000 C CNN
 F 2 "" H 4450 1000 50  0001 C CNN
@@
 $EndComp
 $Comp
-L power:GND #PWR?
+L power:GND #PWR0106
 U 1 1 5E24590D
 P 4450 2450
-F 0 "#PWR?" H 4450 2200 50  0001 C CNN
+F 0 "#PWR0106" H 4450 2200 50  0001 C CNN
 F 1 "GND" H 4455 2277 50  0000 C CNN
 F 2 "" H 4450 2450 50  0001 C CNN
@@
 $EndComp
 $Comp
-L power:+5V #PWR?
+L power:+5V #PWR0107
 U 1 1 5E247C0D
 P 6200 1000
-F 0 "#PWR?" H 6200 850 50  0001 C CNN
+F 0 "#PWR0107" H 6200 850 50  0001 C CNN
 F 1 "+5V" H 6215 1173 50  0000 C CNN
 F 2 "" H 6200 1000 50  0001 C CNN
@@
 $EndComp
 $Comp
-L power:GND #PWR?
+L power:GND #PWR0108
 U 1 1 5E247C19
 P 6200 2450
-F 0 "#PWR?" H 6200 2200 50  0001 C CNN
+F 0 "#PWR0108" H 6200 2200 50  0001 C CNN
 F 1 "GND" H 6205 2277 50  0000 C CNN
 F 2 "" H 6200 2450 50  0001 C CNN
@@
 F 0 "MAX6675" H 5280 3542 50  0000 L CNN
 F 1 "Conn_01x05" H 5280 3451 50  0000 L CNN
-F 2 "Connector_PinHeader_2.00mm:PinHeader_1x05_P2.00mm_Vertical" H 5200 3500 50  0001 C CNN
+F 2 "Connector_PinHeader_2.54mm:PinHeader_1x05_P2.54mm_Vertical" H 5200 3500 50  0001 C CNN
 F 3 "~" H 5200 3500 50  0001 C CNN
 	1    5200 3500
@@
 	4750 3700 5000 3700
 $Comp
-L power:GND #PWR?
+L power:GND #PWR0109
 U 1 1 5E2B4535
 P 4300 3350
-F 0 "#PWR?" H 4300 3100 50  0001 C CNN
+F 0 "#PWR0109" H 4300 3100 50  0001 C CNN
 F 1 "GND" H 4305 3177 50  0000 C CNN
 F 2 "" H 4300 3350 50  0001 C CNN
@@
 	4300 3300 5000 3300
 $Comp
-L power:+5V #PWR?
+L power:+5V #PWR0110
 U 1 1 5E2B8FFC
 P 4700 3400
-F 0 "#PWR?" H 4700 3250 50  0001 C CNN
+F 0 "#PWR0110" H 4700 3250 50  0001 C CNN
 F 1 "+5V" V 4715 3528 50  0000 L CNN
 F 2 "" H 4700 3400 50  0001 C CNN
@@
 Wire Wire Line
 	3000 3400 3600 3400
+Wire Notes Line
+	11200 3450 11200 500
+$Comp
+L Connector_Generic:Conn_01x02 power_ctrl1
+U 1 1 5E3615C0
+P 6450 4500
+F 0 "power_ctrl1" H 6530 4492 50  0000 L CNN
+F 1 "Conn_01x02" H 6530 4401 50  0000 L CNN
+F 2 "TerminalBlock:TerminalBlock_Altech_AK300-2_P5.00mm" H 6450 4500 50  0001 C CNN
+F 3 "~" H 6450 4500 50  0001 C CNN
+	1    6450 4500
+	1    0    0    -1
+$EndComp
+Text Label 6200 4500 2    60   ~ 0
+8
+$Comp
+L Connector_Generic:Conn_01x04 i2c1
+U 1 1 5E389CA3
+P 5000 4400
+F 0 "i2c1" H 5080 4346 50  0000 L CNN
+F 1 "I2C" H 5080 4301 50  0001 L CNN
+F 2 "Connector_PinHeader_2.54mm:PinHeader_1x04_P2.54mm_Vertical" H 5000 4400 50  0001 C CNN
+F 3 "~" H 5000 4400 50  0001 C CNN
+	1    5000 4400
+	1    0    0    -1
+$EndComp
+$Comp
+L power:GND #PWR0111
+U 1 1 5E38EE1A
+P 4100 4350
+F 0 "#PWR0111" H 4100 4100 50  0001 C CNN
+F 1 "GND" H 4105 4177 50  0000 C CNN
+F 2 "" H 4100 4350 50  0001 C CNN
+F 3 "" H 4100 4350 50  0001 C CNN
+	1    4100 4350
+	1    0    0    -1
+$EndComp
+Wire Wire Line
+	4100 4300 4100 4350
+Wire Wire Line
+	4100 4300 4800 4300
+$Comp
+L power:+5V #PWR0112
+U 1 1 5E38EE22
+P 4500 4400
+F 0 "#PWR0112" H 4500 4250 50  0001 C CNN
+F 1 "+5V" V 4515 4528 50  0000 L CNN
+F 2 "" H 4500 4400 50  0001 C CNN
+F 3 "" H 4500 4400 50  0001 C CNN
+	1    4500 4400
+	0    -1   -1   0
+$EndComp
+Wire Wire Line
+	4800 4400 4500 4400
+Text Label 4450 4500 0    60   ~ 0
+A4(SDA)
+Text Label 4450 4600 0    60   ~ 0
+A5(SCL)
+Wire Wire Line
+	4450 4500 4800 4500
+Wire Wire Line
+	4450 4600 4800 4600
+$Comp
+L power:GND #PWR?
+U 1 1 5E3D22C6
+P 6200 4650
+F 0 "#PWR?" H 6200 4400 50  0001 C CNN
+F 1 "GND" H 6205 4477 50  0000 C CNN
+F 2 "" H 6200 4650 50  0001 C CNN
+F 3 "" H 6200 4650 50  0001 C CNN
+	1    6200 4650
+	1    0    0    -1
+$EndComp
+Wire Wire Line
+	6200 4650 6200 4600
+Wire Wire Line
+	6200 4600 6250 4600
+Wire Wire Line
+	6200 4500 6250 4500
 $EndSCHEMATC

Commit message: ...
Connections:
- net L7_collector: now reaches L7.1 (K), T_L7.1 (C)
- net L7_base: now reaches R_B_L7.1, T_L7.2 (B)
- net L7_emitter: now reaches R_E_L7.1, T_L7.3 (E)
- net L6_collector: now reaches L6.1 (K), T_L6.1 (C)
- net L6_base: now reaches R_B_L6.1, T_L6.2 (B)
- net L6_emitter: now reaches R_E_L6.1, T_L6.3 (E)
- net L5_collector: now reaches L5.1 (K), T_L5.1 (C)
- net L5_base: now reaches R_B_L5.1, T_L5.2 (B)
- net L5_emitter: now reaches R_E_L5.1, T_L5.3 (E)
Changed lines of the file:
@@
 Connection ~ 7550 2500
-$Comp
-L Device:LED L7
-U 1 1 5E1DD584
-P 2550 1250
-F 0 "L7" V 2589 1133 50  0000 R CNN
-F 1 "LED" V 2498 1133 50  0000 R CNN
-F 2 "LED_THT:LED_D3.0mm" H 2550 1250 50  0001 C CNN
-F 3 "~" H 2550 1250 50  0001 C CNN
-	1    2550 1250
-	0    -1   -1   0
-$EndComp
-$Comp
-L power:+5V #PWR0103
-U 1 1 5E1DD58A
-P 2550 1000
-F 0 "#PWR0103" H 2550 850 50  0001 C CNN
-F 1 "+5V" H 2565 1173 50  0000 C CNN
-F 2 "" H 2550 1000 50  0001 C CNN
-F 3 "" H 2550 1000 50  0001 C CNN
-	1    2550 1000
-	1    0    0    -1
-$EndComp
 $Comp
 L Transistor_BJT:BC337 T_L7
@@
 F 3 "https://diotec.com/tl_files/diotec/files/pdf/datasheets/bc337.pdf" H 2450 1750 50  0001 L CNN
 	1    2450 1750
-	1    0    0    -1
-$EndComp
-$Comp
-L power:GND #PWR0104
-U 1 1 5E1DD596
-P 2550 2450
-F 0 "#PWR0104" H 2550 2200 50  0001 C CNN
-F 1 "GND" H 2555 2277 50  0000 C CNN
-F 2 "" H 2550 2450 50  0001 C CNN
-F 3 "" H 2550 2450 50  0001 C CNN
-	1    2550 2450
-	1    0    0    -1
-$EndComp
-$Comp
-L Device:R R_E_L7
-U 1 1 5E1DD59C
-P 2550 2200
-F 0 "R_E_L7" H 2620 2246 50  0000 L CNN
-F 1 "500" H 2620 2155 50  0000 L CNN
-F 2 "Resistor_SMD:R_0805_2012Metric" V 2480 2200 50  0001 C CNN
-F 3 "~" H 2550 2200 50  0001 C CNN
-	1    2550 2200
 	1    0    0    -1
 $EndComp
@@
 	0    1    1    0
 $EndComp
-Wire Wire Line
-	2550 1400 2550 1550
-Wire Wire Line
-	2550 1950 2550 2050
-Wire Wire Line
-	2550 2350 2550 2450
-Wire Wire Line
-	2550 1000 2550 1100
 Wire Wire Line
 	2100 1750 2250 1750
@@
 	4450 4600 4800 4600
 $Comp
-L power:GND #PWR?
+L power:GND #PWR0113
 U 1 1 5E3D22C6
 P 6200 4650
-F 0 "#PWR?" H 6200 4400 50  0001 C CNN
+F 0 "#PWR0113" H 6200 4400 50  0001 C CNN
 F 1 "GND" H 6205 4477 50  0000 C CNN
 F 2 "" H 6200 4650 50  0001 C CNN
@@
 Wire Wire Line
 	6200 4500 6250 4500
+Wire Wire Line
+	2550 1000 2550 1100
+Wire Wire Line
+	2550 1400 2550 1550
+$Comp
+L power:+5V #PWR0103
+U 1 1 5E1DD58A
+P 2550 1000
+F 0 "#PWR0103" H 2550 850 50  0001 C CNN
+F 1 "+5V" H 2565 1173 50  0000 C CNN
+F 2 "" H 2550 1000 50  0001 C CNN
+F 3 "" H 2550 1000 50  0001 C CNN
+	1    2550 1000
+	1    0    0    -1
+$EndComp
+$Comp
+L Device:LED L7
+U 1 1 5E1DD584
+P 2550 1250
+F 0 "L7" V 2589 1133 50  0000 R CNN
+F 1 "LED" V 2498 1133 50  0000 R CNN
+F 2 "LED_THT:LED_D3.0mm" H 2550 1250 50  0001 C CNN
+F 3 "~" H 2550 1250 50  0001 C CNN
+	1    2550 1250
+	0    -1   -1   0
+$EndComp
+Wire Wire Line
+	2550 2350 2550 2450
+Wire Wire Line
+	2550 1950 2550 2050
+$Comp
+L Device:R R_E_L7
+U 1 1 5E1DD59C
+P 2550 2200
+F 0 "R_E_L7" H 2620 2246 50  0000 L CNN
+F 1 "500" H 2620 2155 50  0000 L CNN
+F 2 "Resistor_SMD:R_0805_2012Metric" V 2480 2200 50  0001 C CNN
+F 3 "~" H 2550 2200 50  0001 C CNN
+	1    2550 2200
+	1    0    0    -1
+$EndComp
+$Comp
+L power:GND #PWR0104
+U 1 1 5E1DD596
+P 2550 2450
+F 0 "#PWR0104" H 2550 2200 50  0001 C CNN
+F 1 "GND" H 2555 2277 50  0000 C CNN
+F 2 "" H 2550 2450 50  0001 C CNN
+F 3 "" H 2550 2450 50  0001 C CNN
+	1    2550 2450
+	1    0    0    -1
+$EndComp
+Text Label 2550 1500 0    50   ~ 0
+L7_collector
+Text Label 2550 2050 0    50   ~ 0
+L7_emitter
+Text Label 2100 1750 0    50   ~ 0
+L7_base
+Text Label 4450 1550 0    50   ~ 0
+L6_collector
+Text Label 4450 2050 0    50   ~ 0
+L6_emitter
+Text Label 4000 1750 0    50   ~ 0
+L6_base
+Text Label 6200 1550 0    50   ~ 0
+L5_collector
+Text Label 6200 2050 0    50   ~ 0
+L5_emitter
+Text Label 5750 1750 0    50   ~ 0
+L5_base
+Text Label 2550 2450 0    50   ~ 0
+GND
+Text Label 4450 2450 0    50   ~ 0
+GND
+Text Label 6200 2450 0    50   ~ 0
+GND
+Text Label 7550 2250 0    50   ~ 0
++5V
+Text Label 6200 1050 0    50   ~ 0
++5V
+Text Label 4450 1100 0    50   ~ 0
++5V
+Text Label 2550 1050 0    50   ~ 0
++5V
+Text Label 4300 3300 0    50   ~ 0
+GND
+Text Label 4100 4300 0    50   ~ 0
+GND
+Text Label 7550 3200 0    50   ~ 0
+GND
 $EndSCHEMATC
